Commit message: SLAM temps reel (slam_toolbox) + nettoyage du scan lidar
- Fini la carte figee et l'arene virtuelle : slam_toolbox (async) construit la
  carte EN ROULANT et publie map->odom. map_server et map_odom_bridge retires
  de start_nav.sh. Sauvegarde/rechargement de carte : a faire plus tard.
- scan_fix.py (/scan_raw -> /scan) resout DEUX defauts qui cassaient tout :
  1) le N10 sort 449/450/451 rayons selon les tours -> slam_toolbox rejetait
     ~6% des scans ("expected 449") -> reechantillonnage a 450 points fixes.
  2) le lidar VOYAIT LE ROBOT (montants/antennes a 28-48 cm, 49 rayons) :
     obstacles permanents colles au chassis -> nav2 se croyait encercle et
     refusait de planifier. 3 secteurs masques (233-250, 261-280, 282-311 deg),
     seuil de distance par secteur pour garder les vrais obstacles au-dela.
     Verifie : 49 -> 0 echo parasite.
- detect_self.py : detecte automatiquement ces secteurs (echos a variance
  quasi nulle et proches, robot immobile) -> a relancer si le chassis change.
- TF lidar remise a yaw=0 : le retournement du sens de marche avait ete
  compense a tort (le lidar regarde deja le nouvel avant) -> scans en miroir.
- nav.rviz : arene retiree, carte SLAM + scan + costmap locale.
- URDF refait d'apres photos : base bois ronde, roues pneus blancs, 4 montants,
  plateau alu, lidar, batterie bleue, boitier Jetson.

Co-Authored-By: Claude Opus 5 <noreply@anthropic.com>

File: ros2/mowbot.urdf (robot description, URDF)
Before this commit: robot mowbot, 11 links, 10 joints
Links:
- removed link bac
- removed link bac_bord
- removed link caster_front
- removed link liege
- added link battery; visual box size=0.21 0.09 0.075
- added link caster_rear; visual cylinder length=0.022 radius=0.032
- added link deck; visual box size=0.34 0.32 0.005
- added link jetson; visual box size=0.11 0.09 0.045
- added link lidar_body; visual cylinder length=0.048 radius=0.038
- added link post_fl; visual box size=0.04 0.04 0.27
- added link post_fr; visual box size=0.04 0.04 0.27
- added link post_rl; visual box size=0.04 0.04 0.27
- added link post_rr; visual box size=0.04 0.04 0.27
- link base_link: geometry visual cylinder length=0.018 radius=0.22
- link electronics: geometry visual box size=0.13 0.10 0.035
- link front_marker: geometry visual box size=0.05 0.02 0.012
- link hub_left: geometry visual cylinder length=0.048 radius=0.042
- link hub_right: geometry visual cylinder length=0.048 radius=0.042
Joints:
- removed joint bac_to_bord
- removed joint bac_to_liege
- removed joint base_to_bac
- added joint base_to_battery: type fixed, parent base_link, child battery, origin xyz=-0.02 0.05 0.027 rpy=0 0 0.15
- added joint base_to_deck: type fixed, parent base_link, child deck, origin xyz=0.02 0 0.262
- added joint deck_to_jetson: type fixed, parent base_link, child jetson, origin xyz=-0.06 -0.06 0.287 rpy=0 0 0.1
- added joint deck_to_lidar: type fixed, parent base_link, child lidar_body, origin xyz=0.10 0 0.288
- added joint j_post_fl: type fixed, parent base_link, child post_fl, origin xyz=0.13 0.12 0.125
- added joint j_post_fr: type fixed, parent base_link, child post_fr, origin xyz=0.13 -0.12 0.125
- added joint j_post_rl: type fixed, parent base_link, child post_rl, origin xyz=-0.10 0.12 0.125
- added joint j_post_rr: type fixed, parent base_link, child post_rr, origin xyz=-0.10 -0.12 0.125
- joint base_to_caster: child caster_front -> caster_rear; origin xyz=0.19 0 -0.035 rpy=0 0 0 -> xyz=-0.17 0 -0.043 rpy=0 0 0
- joint base_to_electronics: origin xyz=-0.05 -0.06 0.02 rpy=0 0 0.3 -> xyz=0.06 -0.09 0.007 rpy=0 0 -0.2
- joint base_to_front: origin xyz=0.21 0 -0.01 rpy=0 0 0 -> xyz=0.205 0 -0.012
- joint wheel_left_hub: origin xyz=0 0 0 rpy=0 0 0 -> xyz=0 0 0
- joint wheel_right_hub: origin xyz=0 0 0 rpy=0 0 0 -> xyz=0 0 0
