Commit message: geometrie reelle : entraxe 0.48 m et debord arriere de 10 cm
Deux mesures fournies par l'utilisateur qui invalidaient des hypotheses de base.

1. ENTRAXE 0.48 m (firmware, robot 24 V uniquement)
   TRACK_WIDTH_M etait reste a 0.59, valeur heritee du chassis 12 V. La
   cinematique inverse (v = w*L/2) faisait donc sur-tourner le robot de ~23 %
   sur chaque consigne angulaire : nav2 demandait 0.20 rad/s, le robot
   tournait a 0.246. Le cap etant fourni par le gyro, l'odometrie masquait
   l'erreur — seule la COMMANDE etait fausse, d'ou des virages toujours trop
   serres et des corrections en boucle.

2. DEBORD ARRIERE +10 cm : le robot n'est plus un disque centre
   nav2 le modelisait en robot_radius 0.22. Or il fait 0.24 devant, 0.34
   derriere et 0.265 de demi-largeur. Consequences : l'arriere n'etait PAS
   protege (grave, la marche arriere venant d'etre autorisee) et les cotes
   etaient sous-estimes de 4 cm. Remplace par le contour polygonal reel a
   8 points sur les deux costmaps — plus juste que le disque englobant de
   0.34, qui aurait ajoute 12 cm de bourrelet inutile a l'avant.

Corollaires de la taille reelle :
- lookahead 0.20 -> 0.35 m : a 0.20 le point de poursuite tombait DANS le
  robot (avant a 0.24) -> braquage permanent, oscillations, blocages.
- tolerance d'arrivee 0.08 -> 0.12 m : viser 8 cm avec un robot de 58 cm a
  0.048 m/s faisait durer le dernier centimetre plus que le trajet.
- costmap local 2x2 -> 3x3 m : marge de manoeuvre pour les marches arriere.
- URDF : roues a +/-0.24, plaque arriere ajoutee.

NON VALIDE AU SOL : les moteurs ne repondent plus (0 tick a pleine consigne)
alors que micro-ROS et /odom fonctionnent -> alimentation 24 V a verifier.

Co-Authored-By: Claude Opus 5 <noreply@anthropic.com>

File: robot/config/mowbot.urdf (robot description, URDF)
Before this commit: robot mowbot, 16 links, 15 joints
Links:
- added link rear_ext; visual box size=0.10 0.30 0.018
Joints:
- added joint base_to_rear_ext: type fixed, parent base_link, child rear_ext, origin xyz=-0.27 0 -0.02
- joint base_to_wheel_left: origin xyz=0 0.215 0 rpy=0 0 0 -> xyz=0 0.24 0 rpy=0 0 0
- joint base_to_wheel_right: origin xyz=0 -0.215 0 rpy=0 0 0 -> xyz=0 -0.24 0 rpy=0 0 0

Commit message: languette arriere reelle (5 cm), inflation 5 cm, et bascule des services
GEOMETRIE — la "rallonge arriere" etait fausse : ce n'est pas une plaque de
10x30 cm sur tout l'arriere mais une petite languette en bois de ~5 cm de
debord sur ~15 cm de large, celle qui porte la roulette folle (verifie sur
photo). URDF et footprint nav2 corriges : contour a 10 points qui epouse le
disque (r=0.22), les pneus (point le plus large, +/-0.26) et la languette
(-0.27 sur 15 cm). Le disque englobant equivalent aurait fait 0.27 partout,
soit 5 cm de bourrelet inutile tout autour.

INFLATION 0.10 -> 0.05 (demande utilisateur : "ca bloque de temps en temps
pour rien"). Justifie ici : le footprint decrit deja la taille reelle, et
l'inflation ne sert plus qu'a lisser la trajectoire.

BASCULE DES SERVICES — la reorganisation n'avait jamais ete activee sur la
Jetson : les 9 services systemd pointaient encore vers les anciens scripts
de /home/nvidia/, qui lisaient /home/nvidia/nav2_params.yaml. Autrement dit
TOUS les reglages ecrits dans ~/mowbot/config/ depuis la reorganisation
etaient ignores — la navigation tournait encore a desired_linear_vel 0.035
avec robot_radius 0.24. Deux arborescences divergeaient en silence.
install.sh relance -> les services pointent maintenant vers ~/mowbot/bin/.
Anciens scripts conserves dans ~/legacy_scripts_backup/ (61 fichiers).
Verifie : le footprint publie a bien 10 points, donc la bonne config est lue.

BUG run_description.sh — passer l'URDF en argument
(-p robot_description:="$(cat ...)") casse l'analyse des arguments rclcpp des
qu'il contient des sauts de ligne : le noeud redemarrait en boucle sans
jamais publier le modele. Remplace par nodes/description.launch.py, qui lit
le fichier via $MOWBOT_CONFIG (portable, pas de chemin en dur comme l'ancien
/home/nvidia/description.launch.py).

Verifie depuis le PC : arbre TF complet, rear_ext presente, scan a 10 Hz.

Co-Authored-By: Claude Opus 5 <noreply@anthropic.com>

File: robot/config/mowbot.urdf (robot description, URDF)
Before this commit: robot mowbot, 17 links, 16 joints
Links:
- link rear_ext: geometry visual box size=0.05 0.15 0.018
Joints:
- joint base_to_rear_ext: origin xyz=-0.27 0 -0.02 -> xyz=-0.245 0 -0.02

Commit message: Jetson en conteneur Jazzy : arret propre des services, TF sans retard, lidar natif
Suite de la mise en service du Xavier NX. Quatre problemes distincts, chacun
avec sa mesure.

1. LES TF AVAIENT UNE SECONDE DE RETARD SUR LES SCANS, cause reelle de tout ce
   qu'on observait -- slam_toolbox jetant TOUS les scans ("queue is full"),
   aucune carte, et les "extrapolation into the future" de RViz sur `odom`
   comme sur `laser_link`. L'EKF a 30 Hz ne tenait pas la cadence sur cette
   machine. Passe a 15 Hz : /odom arrive a 10 Hz et l'IMU a 20, inutile d'aller
   plus vite.
     avant : requested ...489.111, latest ...488.07  -> 1040 ms
     apres : requested ...302.639, latest ...302.62  ->   19 ms
     /map republie a 1.22 Hz, rejets SLAM tombes a 8

2. ARRET DES SERVICES DANS LE CONTENEUR. `docker exec` laisse le processus
   survivre a l'arret de l'unite : chaque restart empilait une instance (deux
   slam_toolbox sur la meme TF, trois planner_server, charge 54). TROIS
   tentatives avant d'y arriver, et les deux premieres etaient fausses :
     - pkill sur le chemin du script : inoperant, tous les run_*.sh finissent
       par `exec` et le bash est remplace ;
     - `echo $$` depuis ExecStart : systemd lit `$$` comme un `$` litteral, les
       fichiers de PID contenaient donc un `$`. Et les lignes etaient AJOUTEES
       EN FIN DE FICHIER, donc dans [Install], ou systemd ignore les cles
       Exec* -- l'ExecStop n'a jamais existe ;
     - `$(cat fichier)` dans l'unite : systemd ne fait aucune substitution de
       commande, "bad unit file setting", TOUS les services refusaient de
       demarrer.
   Version retenue : bin/ct_stop.sh porte la logique, l'unite ne passe que deux
   arguments sans caractere special, et le PID est ecrit par mowbot_env.sh en
   shell ordinaire. Chaque unite est verifiee par `systemd-analyze verify`.

3. DRIVER LIDAR NATIF compile dans le conteneur, sous $MOWBOT_HOME pour
   survivre aux redemarrages (seul dossier monte). 7.4 % d'un coeur contre 17.5
   pour le noeud Python. Le correctif pthread de log_module.h est applique
   automatiquement. Un ancien ld14_node.py tenait ENCORE /dev/ttyUSB0 en meme
   temps que le natif : les deux se volaient les octets.

4. POSITION DU LIDAR : -0.16 m et non -0.10, MESUREE au metre entre l'axe des
   roues et le centre du lidar, et recoupee independamment a partir du scan
   (-0.167). L'URDF dessinait meme le lidar a +0.10 pendant que la TF publiait
   -0.10 : 20 cm d'ecart de part et d'autre du centre. Les deux fichiers se
   renvoient desormais l'un a l'autre en commentaire.

Aussi : mode 15W/6CORE au lieu de 10W (deux coeurs etaient desactives), journal
systemd rendu persistant (un reset precedent est reste indiagnosticable), et
mesure des cadences par rclpy -- `ros2 topic hz` ne produit rien dans ce
contexte et faisait croire que TOUS les topics etaient muets.

Co-Authored-By: Claude Opus 5 <noreply@anthropic.com>

File: robot/config/mowbot.urdf (robot description, URDF)
Before this commit: robot mowbot, 17 links, 16 joints
Joints:
- joint base_to_wheel_left: origin xyz=0 0.24 0 rpy=0 0 0 -> xyz=0 0.23035 0 rpy=0 0 0
- joint base_to_wheel_right: origin xyz=0 -0.24 0 rpy=0 0 0 -> xyz=0 -0.23035 0 rpy=0 0 0
- joint deck_to_lidar: origin xyz=0.10 0 0.288 -> xyz=-0.16 0 0.288

Commit message: Alleger le SLAM, et corriger la geometrie AFFICHEE des roues
SLAM. Sur le Jetson, /map etait tombe a 0,24 Hz et la TF map->odom accusait
CINQ SECONDES de retard : nav2 echouait alors sur chaque but ("Transform data
too old when converting from odom to map", "Unable to transform robot pose into
global plan's frame"). Trois reglages, tous du meme ordre -- ne pas faire
calculer au SLAM ce que la navigation n'exploite pas :
  . resolution 0.03 -> 0.05 : a 3 cm la carte comptait QUATRE FOIS plus de
    cellules a calculer et republier, alors que la costmap tourne a 4 cm et que
    le robot fait 50 cm de large ;
  . map_update_interval 1.0 -> 2.0 : republier la carte entiere coute cher et
    elle n'a pas besoin d'etre fraiche a la seconde ;
  . max_laser_range 12.0 -> 8.0 : portee REELLE du LD14. Annoncer 12 faisait
    traiter des cellules que le capteur ne voit jamais.

ROUES. Plainte constatee : la roue TOUCHAIT un obstacle dans RViz alors qu'elle
en etait a 1 cm dans la realite. Les roues dessinees sont donc rentrees de 1 cm
(0.23035 -> 0.22035) et le rayon du plateau suit (0.22 -> 0.2429 = bord
exterieur des roues dessinees). L'ancienne valeur faisait DEPASSER les roues du
plateau a l'ecran, ce qui laissait croire a une erreur de geometrie.

CE FICHIER NE SERT QU'A L'AFFICHAGE : il n'entre ni dans la cinematique ni dans
la detection de collision, qui utilise le footprint de nav2_params.yaml. Trois
allers-retours ont ete perdus a modifier le footprint de collision alors que la
plainte portait sur le DESSIN.

Co-Authored-By: Claude Opus 5 <noreply@anthropic.com>

File: robot/config/mowbot.urdf (robot description, URDF)
Before this commit: robot mowbot, 17 links, 16 joints
Links:
- link base_link: geometry visual cylinder length=0.018 radius=0.2429
Joints:
- joint base_to_wheel_left: origin xyz=0 0.23035 0 rpy=0 0 0 -> xyz=0 0.22035 0 rpy=0 0 0
- joint base_to_wheel_right: origin xyz=0 -0.23035 0 rpy=0 0 0 -> xyz=0 -0.22035 0 rpy=0 0 0

Commit message: URDF : la roulette folle devient la roue directrice, et deux commentaires faux
Le modele decrivait encore une roulette folle a -0,17 alors que la roue
directrice, mesuree, est a -0,36. Meme mecanisme que le tableau de cablage du
README qui annonçait huit broches fausses sur dix : une cote dupliquee dont
une copie a vieilli.

  caster_rear (-0,17)  ->  steer_wheel (-0,36)
  bras arriere : boite de 0,05 m a -0,245  ->  0,16 m a -0,29

DEUX COMMENTAIRES ETAIENT FAUX, et l'un a failli couter cher

L'en-tete affirmait "x = AVANT (cote lidar)". C'est l'inverse : front_marker
est a +0,205 et les montants avant a +0,13, donc +x est bien l'avant, mais le
LIDAR est a -0,16, c'est-a-dire A L'ARRIERE. Cette phrase m'a fait douter du
cote ou se trouve la roue directrice, alors que ce doute decide du SIGNE du
modele de direction. Corrigee, avec la preuve qui la contredit.

Le commentaire du joint lidar annonçait encore "x = -0.10" alors que la valeur
du fichier est -0.16 depuis sa correction. Aligne.

DEDUIT ET NON MESURE, signale comme tel dans le fichier : la longueur du bras
arriere (calculee entre le bord du plateau et la roue) et le rayon de la roue
directrice, repris de l'ancienne roulette. Si ce rayon change, corriger le
rayon ET le z ensemble, sinon la roue flotte ou s'enfonce dans le sol.

Le joint reste FIXE : l'angle de braquage n'est pas anime. L'animer demanderait
un joint_states alimente par le delta commande du firmware. Le modele n'a aucun
effet sur la navigation, il ne sert qu'a l'affichage -- mais un dessin faux
fait chercher des pannes inexistantes.

Verifie : XML bien forme, plus aucune mention de caster dans le depot, et
l'ecart steer_wheel - lidar_body vaut exactement les 0,200 m mesures.

Co-Authored-By: Claude Opus 5 (1M context) <noreply@anthropic.com>

File: robot/config/mowbot.urdf (robot description, URDF)
Before this commit: robot mowbot, 17 links, 16 joints
Links:
- removed link caster_rear
- added link steer_wheel; visual cylinder length=0.022 radius=0.032
- link rear_ext: geometry visual box size=0.16 0.15 0.018
Joints:
- removed joint base_to_caster
- added joint base_to_steer_wheel: type fixed, parent base_link, child steer_wheel, origin xyz=-0.36 0 -0.043 rpy=0 0 0
- joint base_to_rear_ext: origin xyz=-0.245 0 -0.02 -> xyz=-0.29 0 -0.02

Commit message: URDF : la roue directrice TOURNE enfin dans RViz
Elle etait dessinee au bon endroit mais figee : mowbot.urdf n'avait que des
joints fixes, et je l'avais laissee fixe faute de source pour l'angle. La
source existait pourtant.

LE FIRMWARE NE PUBLIE PAS L'ANGLE DU SERVO (servo RC sans retour), MAIS SON
ODOMETRIE LE CONTIENT :
    w = v * tan(delta) / x_s   (modele bicyclette, kin_ackermann.c)
    donc delta = atan(w * x_s / v)
Reconstruction verifiee EXACTE sur 25 cas, marche arriere comprise : ecart max
2,8e-17 rad. C'est l'angle COMMANDE, pas le reel -- personne ne connait le
second sans retour de position, et la mesure du jour montre justement que le
reel est plus faible. RViz montre donc ce que le firmware DEMANDE.

  mowbot.urdf        base_to_steer_wheel (fixed) devient deux joints :
                     base_to_steer_pivot (fixed, la position) + steer_joint
                     (revolute, axe z, bornes +-STEER_MAX_RAD). C'est ce
                     decoupage qui permet la rotation.
  nodes/steer_state.py  publie /joint_states a 20 Hz. A l'arret (v au
                     denominateur) il GARDE le dernier angle : le servo tient
                     sa position, c'est fidele au materiel. Geometrie lue de
                     config/ackerbot_geometry.env, rien en dur ; fichier absent
                     -> joint publie a ZERO avec un avertissement, car sans
                     /joint_states robot_state_publisher n'emet pas du tout la
                     TF de la roue et elle disparait du modele. Un angle faux
                     serait pire qu'un angle nul.
  description.launch.py  lance le publieur A COTE du modele, et seulement si
                     l'URDF contient steer_joint : un chassis diffdrive ne
                     lance rien de plus. Un URDF a joint mobile sans publieur
                     est incomplet, les deux vont ensemble.
  gen_ackerbot_geometry.py  exporte ACKERBOT_STEER_MAX_RAD, pour que la borne
                     du joint et l'ecretage du noeud viennent de la MEME source
                     que le rayon de braquage.

VERIFIE sur le robot : /joint_states publie a 20,07 Hz par /steer_state, joint
steer_joint present, et le noeud annonce au demarrage "x_s=-0.360 m (derriere
l'essieu), butee 45.0 deg".

A SAVOIR EN REGARDANT RVIZ : la roue est DERRIERE l'essieu moteur, donc pour
virer a gauche elle pointe a DROITE. Un braquage oppose au virage est NORMAL
sur ce chassis -- c'est ecrit dans le commentaire du joint.

Co-Authored-By: Claude Opus 5 (1M context) <noreply@anthropic.com>

File: robot/config/mowbot.urdf (robot description, URDF)
Before this commit: robot mowbot, 17 links, 16 joints
Links:
- added link steer_pivot
Joints:
- removed joint base_to_steer_wheel
- added joint base_to_steer_pivot: type fixed, parent base_link, child steer_pivot, origin xyz=-0.36 0 -0.043 rpy=0 0 0
- added joint steer_joint: type revolute, parent steer_pivot, child steer_wheel, origin xyz=0 0 0 rpy=0 0 0, axis 0 0 1, limit lower=-0.7854 upper=0.7854 effort=1.0 velocity=3.0

Commit message: Sens de marche INVERSE : l'avant du robot est le cote de la roue directrice
"le servo moteur tourne du mauvais cote" -- repete plusieurs fois, et j'ai
cherche l'erreur au mauvais endroit. Le diagnostic est venu de cette phrase :
"le servo tourne bien a gauche mais le robot roule en ARRIERE et non en
direction du servo".

RIEN N'ETAIT CASSE. Le logiciel appelait "avant" le cote OPPOSE au servo, la
configuration etait parfaitement coherente avec elle-meme -- c'est pourquoi le
gyroscope concordait avec l'odometrie 17 fois sur 17 -- mais elle etait a
l'envers du robot reel. D'ou le braquage vecu comme inverse : avec la roue
placee derriere, le firmware la fait pointer a droite pour virer a gauche.
Avec la roue DEVANT, c'est le comportement d'une voiture ordinaire.

CE QUI A CHANGE, d'un seul tenant (base_link tourne de 180 deg autour de z) :

  robot.h    STEER_X_M -0.36 -> +0.36. Broches moteur et encodeurs ECHANGEES
             (le canal 22/23 devient la roue DROITE, 20/21 la GAUCHE) et les
             DEUX moteurs inverses. Les drapeaux d'encodeur gardent leurs
             valeurs : l'echange gauche/droite et l'inversion du sens de
             marche se compensent exactement -- explique en commentaire.
  mowbot.urdf  modele entier en miroir (x et y). Etiquettes avant/arriere et
             gauche/droite REATTRIBUEES d'apres les positions obtenues, sinon
             on recreait exactement la confusion qui a coute cette soiree.
             rear_ext devient steer_arm. front_marker n'est PAS mis en miroir :
             repere d'affichage, il doit rester a l'avant.
  run_tf.sh  MOWBOT_LIDAR_X -0.16 -> +0.16 : le lidar passe EN TETE du sens de
             marche, ce qui est un gain reel pour la detection d'obstacles.
  nav2       empreinte en miroir : le long cote (0.40, le bras de direction)
             est desormais a l'AVANT.

LE ROBOT DEVIENT UN TRICYCLE CLASSIQUE : roue directrice qui mene, deux roues
motrices derriere. Configuration stable, contrairement a la precedente qui
etait celle d'un chariot elevateur (essieu directeur qui traine).
Ce que l'inversion ne change PAS, verifie : l'anneau balaye en virage est
IDENTIQUE (0,485 m), et le point le plus exterieur reste un coin avant. J'avais
suppose le contraire ; c'etait faux, retourner le repere ne change pas la
geometrie autour du centre de rotation. Ce qui change, c'est que le
debordement de 0,139 m de la roue directrice se produit maintenant DEVANT, la
ou le lidar regarde.

VERIFIE : les trois controleurs compilent, 0 avertissement ; 44 verifications
hotes passent dans les DEUX geometries (le test etait deja parametre par le
signe, il n'a rien coute) ; flashe depuis la Jetson (esptool 4.12, --force pour
la revision v1.3, agent arrete puis relance) ; TF relevees sur le robot :
laser_link +0.160, steer_pivot +0.360, front_marker +0.205, tous du bon cote ;
bt_navigator actif.

NON VERIFIE, ET C'EST LE POINT SENSIBLE : les quatre signes moteur/encodeur
sont DEDUITS, pas mesures. C'est exactement le genre d'echange qui a deja coute
une seance sur robot A. kin_bench_test() teste chaque roue separement contre
son propre encodeur : c'est lui qui doit valider, roues en l'air, avant de
reposer le robot au sol.

ET J'AI REFAIT L'ERREUR DOCUMENTEE TROIS FOIS DANS CE DEPOT : un double tiret
dans un commentaire XML, qui a rendu l'URDF invalide. Detectee par le parseur
tout de suite. Le depot le dit pourtant en toutes lettres.

Co-Authored-By: Claude Opus 5 (1M context) <noreply@anthropic.com>

File: robot/config/mowbot.urdf (robot description, URDF)
Before this commit: robot mowbot, 18 links, 17 joints
Links:
- removed link rear_ext
- added link steer_arm; visual box size=0.16 0.15 0.018
Joints:
- removed joint base_to_rear_ext
- added joint base_to_steer_arm: type fixed, parent base_link, child steer_arm, origin xyz=0.29 0 -0.02
- joint base_to_battery: origin xyz=-0.02 0.05 0.027 rpy=0 0 0.15 -> xyz=0.02 -0.05 0.027 rpy=0 0 0.15
- joint base_to_deck: origin xyz=0.02 0 0.262 -> xyz=-0.02 0 0.262
- joint base_to_electronics: origin xyz=0.06 -0.09 0.007 rpy=0 0 -0.2 -> xyz=-0.06 0.09 0.007 rpy=0 0 -0.2
- joint base_to_steer_pivot: origin xyz=-0.36 0 -0.043 rpy=0 0 0 -> xyz=0.36 0 -0.043 rpy=0 0 0
- joint deck_to_jetson: origin xyz=-0.06 -0.06 0.287 rpy=0 0 0.1 -> xyz=0.06 0.06 0.287 rpy=0 0 0.1
- joint deck_to_lidar: origin xyz=-0.16 0 0.288 -> xyz=0.16 0 0.288
- joint j_post_fl: origin xyz=0.13 0.12 0.125 -> xyz=0.1 0.12 0.125
- joint j_post_fr: origin xyz=0.13 -0.12 0.125 -> xyz=0.1 -0.12 0.125
- joint j_post_rl: origin xyz=-0.10 0.12 0.125 -> xyz=-0.13 0.12 0.125
- joint j_post_rr: origin xyz=-0.10 -0.12 0.125 -> xyz=-0.13 -0.12 0.125
