Commit message: URDF du gros robot : reprendre les noms de reperes que RViz attend
En ecrivant le modele j'ai nomme le repere d'avant "avant". Or pc/odom.rviz du
depot reference "front_marker", le nom historique : la vue affichait donc une
erreur sur un repere introuvable, alors que le modele lui-meme etait sain.
Renommer coutait moins cher que de modifier les vues.

Ajoute aussi "deck" et "lidar_body", presents dans l'ancien modele et
susceptibles d'etre references ailleurs. Ils n'ont aucun role fonctionnel --
c'est de la compatibilite d'affichage, et c'est dit dans le fichier.

Verifie sur le robot apres redemarrage du service : gros.urdf (5774 octets),
et les dix reperes publies sont base_link, chassis, deck, front_marker,
imu_link, laser_link, lidar_body, roue_folle, wheel_left, wheel_right.

Co-Authored-By: Claude Opus 5 (1M context) <noreply@anthropic.com>

File: robot/config/gros.urdf (robot description, URDF)
Before this commit: robot gros, 6 links, 5 joints
Links:
- removed link avant
- added link deck; visual box size=0.60 0.70 0.02
- added link front_marker; visual box size=0.10 0.30 0.04
- added link lidar_body; visual cylinder length=0.05 radius=0.040
Joints:
- removed joint chassis_to_avant
- added joint base_to_deck: type fixed, parent base_link, child deck, origin xyz=0.30 0 0.33 rpy=0 0 0
- added joint base_to_lidar_body: type fixed, parent base_link, child lidar_body, origin xyz=0 0 0.28 rpy=0 0 0
- added joint chassis_to_front_marker: type fixed, parent base_link, child front_marker, origin xyz=0.90 0 0.34 rpy=0 0 0

Commit message: Le modele du gros robot etait illisible : tout blanc et roues noyees
Deux defauts d'affichage, vus sur une capture de RViz.

TOUT SORTAIT EN BLANC. Les materiaux etaient declares au niveau du robot puis
references par nom dans chaque visual -- une forme valide, que RViz n'a pas
reprise ici. Chaque visual porte desormais sa couleur EN LIGNE. 11 couleurs
dans le modele publie, verifiees a la reception.

LES ROUES DISPARAISSAIENT DANS LE CHASSIS. Je l'avais dessine a 0,90 m de large,
la valeur de l'empreinte -- or 0,90 est l'encombrement REEL, ROUES COMPRISES.
Les roues, a +/-0,41 m, se retrouvaient donc a l'interieur de la dalle et n'en
depassaient qu'en haut et en bas. Geometriquement exact, visuellement inutile.
Le chassis est dessine a 0,74 m, les roues ressortent, et l'empreinte nav2 reste
a 0,90 : le dessin sert a comprendre, l'empreinte sert a ne pas heurter.

Valide par check_urdf : "Successfully Parsed XML", base_link a 7 enfants.
Publie sur le robot : 6145 octets, 8 liens, 11 couleurs.

Co-Authored-By: Claude Opus 5 (1M context) <noreply@anthropic.com>

File: robot/config/gros.urdf (robot description, URDF)
Before this commit: robot gros, 8 links, 7 joints
Links:
- link chassis: geometry visual box size=1.15 0.74 0.14
